File: Eagle/AudioSwitch.brd (EAGLE design)
At the start: 15.2 x 24.1 mm, 6 parts, among them U1 2:1_MUX_NC7SZ157P6X

Commit message: update audioboard files
Parts:
- moved R2 6.38 mm to (7.62, 10.8), turned to 180 degrees
- moved R1 1.42 mm to (7.62, 13.3)
- moved U1 0.63 mm to (7.62, 6.99)
Routing:
- net SWITCH: track 20.1 -> 11.4 mm, vias 0 -> 1
- net 0: track 13.4 -> 5.69 mm, vias 0 -> 3
- net VCC: track 39.3 -> 36.5 mm
- net SPDIF_IN_2: track 11.6 -> 12.9 mm
- net SIGNAL_DET: track 4.25 -> 5.39 mm
- net SPDIF_IN_1: track 15.1 -> 15.9 mm
- net TEENSY_SPDIF_IN: track 4.23 -> 4.89 mm
Other:
- board text added: "3v3"
- board text added: "COAX IN"
- board text added: "GND"
- board text added: "OPTICAL IN"
- board text added: "S/PDIF Signal"
- board text added: "Signal Detect"
- board text added: "Switch"
