File: Eagle/AudioBoard.brd (EAGLE design)
At the start: 160 x 100 mm, 5 parts, among them M1 WIRELESS-NRF24L01

Commit message: schematic and board file work.
Parts:
- added R1: 250, resistor:R0805
- added U1: NC7SZ157P6X, MUX_2-1_NC7SZ157P6X:SOIC_Z157P6X_ONS
- moved U$3 96.1 mm to (61.0, 12.7), turned to 180 degrees
- moved U$2 88.8 mm to (31.8, 12.7), turned to 180 degrees
- moved M1 65.9 mm to (35.6, 29.2)
- moved U$1 62.0 mm to (19.1, 36.8), turned to 180 degrees
- moved U$4 43.7 mm to (10.2, 40.6), turned to 180 degrees
Connections:
- removed net VCC: M1.2
- new net CE: M1.3, U$1.5
- new net CSN: M1.4, U$1.9
- new net I2S_DIN: U$1.8
- new net I2S_DOUT: U$1.7
- new net IRQ: M1.8, U$1.16
- new net LED: U$1.3
- new net LRCLK: U$1.20
- new net MCLK: U$1.23
- new net MISO: M1.7, U$1.12
- new net MOSI: M1.6, U$1.11
- new net MUX_SWITCH: U1.6
- new net N$1: U$1.RX
- new net N$11: U$1.10
- new net N$18: U$1.17
- new net N$2: U$1.TX
- new net N$23: U$1.22
- new net N$3: U$1.2
- new net N$5: U$1.4
- new net N$7: U$1.6
- new net S/PDIF-IN: U$1.14, U1.4
- new net S/PDIF-OUT: U$1.15, U$3.SIGNAL
- new net S/PDIF_0_IN: U1.3
- new net S/PDIF_1_IN: R1.1, U$2.SIGNAL, U1.1
- new net SCK: M1.5, U$1.13
- new net SCLK: U$1.21
- new net SGTL_SCL: U$1.19
- new net SGTL_SDA: U$1.18
- new net SIGNAL_DETECT: R1.2
- net 3V3: now also M1.2, U$2.VCC, U$3.VCC, U1.5
- net GND: now also U$2.GND, U$3.GND, U1.2
Other:
- board outline removed

Commit message: schematic and board file work.
Parts:
- removed U$1: TEENSY4.0, Teensy3.2:TEENSY4.0
- added U$5: TEENSY4.0_FULL_IO, Teensy3.2:TEENSY4.0_FULL_IO
- moved R1 23.6 mm to (6.10, 33.1), turned to 180 degrees
- moved M1 7.62 mm to (35.6, 36.8), turned to 90 degrees
- moved U1 2.84 mm to (31.8, 16.5)
- moved U$4 1.27 mm to (10.2, 41.9)
Connections:
- removed net N$1: U$1.RX
- removed net N$11: U$1.10
- removed net N$18: U$1.17
- removed net N$2: U$1.TX
- removed net N$23: U$1.22
- removed net N$3: U$1.2
- removed net N$5: U$1.4
- removed net N$7: U$1.6
- new net N$10: U$5.22
- new net N$16: U$5.17
- new net N$28: U$5.10
- new net N$32: U$5.6
- new net N$34: U$5.4
- new net N$36: U$5.2
- new net N$37: U$5.TX
- new net N$38: U$5.RX
- new net N$42: U$5.26
- new net N$43: U$5.27
- new net N$44: U$5.28
- new net N$45: U$5.29
- new net N$46: U$5.30
- new net N$47: U$5.31
- new net N$48: U$5.32
- new net N$49: U$5.33
- net 3V3: now also U$5.3.3V; no longer U$1.3.3V
- net 5V: now also U$5.VIN; no longer U$1.VIN
- net CE: now also U$5.5; no longer U$1.5
- net CSN: now also U$5.9; no longer U$1.9
- net GND: now also U$5.AGND, U$5.GND, U$5.GND2; no longer U$1.AGND, U$1.GND, U$1.GND2
- net I2S_DIN: now also U$5.8; no longer U$1.8
- net I2S_DOUT: now also U$5.7; no longer U$1.7
- net IRQ: now also U$5.16; no longer U$1.16
- net LED: now also U$5.3; no longer U$1.3
- net LRCLK: now also U$5.20; no longer U$1.20
- net MCLK: now also U$5.23; no longer U$1.23
- net MISO: now also U$5.12; no longer U$1.12
- net MOSI: now also U$5.11; no longer U$1.11
- net MUX_SWITCH: now also U$5.25
- net ON/OFF: now also U$5.ON/OFF; no longer U$1.ON/OFF
- net S/PDIF-IN: now also U$5.14; no longer U$1.14
- net S/PDIF-OUT: now also U$5.15; no longer U$1.15
- net SCK: now also U$5.13; no longer U$1.13
- net SCLK: now also U$5.21; no longer U$1.21
- net SGTL_SCL: now also U$5.19; no longer U$1.19
- net SGTL_SDA: now also U$5.18; no longer U$1.18
- net SIGNAL_DETECT: now also U$5.24

Commit message: updates to eagle files
Parts:
- removed M1: WIRELESS-NRF24L01, NRF24L01:WIRELESS-NRF24L01
- added C1: 0.1u, rcl:C0603K
- added C12, C13: 22pF, SparkFun:0402-CAP
- added C14: 33nF, SparkFun:0402-CAP
- added C15: 2.2nF, SparkFun:0402-CAP
- added C16: 4.7pF, SparkFun:0402-CAP
- added C17: 1.0pF, SparkFun:0402-CAP
- added C18: 1.5pF, SparkFun:0402-CAP
- added C2: 0.1uF, rcl:C0603
- added C3: (no value), rcl:C0603
- added C4, C6, C7, C8: (no value), resistor:C0603
- added C5: 10n, resistor:R0603
- added J1: (no value), SparkFun-Connectors:USB-B-MICRO-SMD_RED_PASTE
- added L1: 47uH, resistor:L2012C
- added L5: 3.9nH, SparkFun:C0402
- added L6: 2.7nH, SparkFun:C0402
- added L7: 8.2nH, SparkFun:C0402
- added Q2: 16MHz, SparkFun:CRYSTAL-SMD-5X3
- added R10: 22K, SparkFun:0402-RES
- added R2, R3: 100, resistor:R0603
- added R4: 8k2, resistor:R0603
- added R5: 330, rcl:R0603
- added R6: 10k, rcl:R0603
- added R9: 1M, SparkFun:0402-RES
- added RECEIVER: S/PDIF-IN, SPDIF:SPDIF-IN
- added TRANSMITTER: S/PDIF-OUT, SPDIF:SPDIF-OUT
- added U$1: 1X3HEADER, 1x2HEADER:1X3HEADER
- added U$6, U$7, U$8: WS2812B, Neopixel WS2812B:WS2812B
- added U$9: 2X4HEADER, 1x2HEADER:2X4HEADER
- added U2: 2:1_MUX_NC7SZ157P6X, AudioSwitch:SOIC_Z157P6X_ONS
- added U3: M74VHC1G125DFT2GSC-88A_ONS-M, AudioSwitch:SC-88A_ONS-M
- added U4: NRF24L01ALT1, Testing:QFN20_ALT1
- added Y2: ANTENNA2SMD5, SparkFun:ANTENNA-CHIP5
- R1: value 250 -> 100; device resistor:R0805 -> resistor:R0603
- U$2: value S/PDIF-IN -> RCA_JACK; device SPDIF:SPDIF-IN -> COAX_SPDIF:RCA_JACK
- U$3: value S/PDIF-OUT -> TEENSY4.0; device SPDIF:SPDIF-OUT -> Teensy3.2:TEENSY4.0
- U$5: value TEENSY4.0_FULL_IO -> WS2812B; device Teensy3.2:TEENSY4.0_FULL_IO -> Neopixel WS2812B:WS2812B
- U1: value NC7SZ157P6X -> SN74HC04_INVERTER; device MUX_2-1_NC7SZ157P6X:SOIC_Z157P6X_ONS -> COAX_SPDIF:NS14
- moved U$3 73.0 mm to (5.08, 59.7), turned to 270 degrees
- moved U$5 36.8 mm to (-17.8, 36.8)
- moved R1 18.7 mm to (24.8, 31.8), turned to 90 degrees
- moved U1 17.8 mm to (33.0, 34.3), turned to 0 degrees
- moved U$2 14.2 mm to (25.4, 25.4)
- moved U$4 5.68 mm to (7.62, 36.8)
Connections:
- removed net N$10: U$5.22
- removed net N$28: U$5.10
- removed net N$32: U$5.6
- removed net N$34: U$5.4
- removed net N$36: U$5.2
- removed net N$37: U$5.TX
- removed net N$38: U$5.RX
- removed net N$42: U$5.26
- removed net N$43: U$5.27
- removed net N$44: U$5.28
- removed net N$45: U$5.29
- removed net N$46: U$5.30
- removed net N$47: U$5.31
- removed net N$48: U$5.32
- removed net N$49: U$5.33
- removed net S/PDIF-IN: U$5.14, U1.4
- removed net S/PDIF_0_IN: U1.3
- removed net S/PDIF_1_IN: R1.1, U$2.SIGNAL, U1.1
- removed net SIGNAL_DETECT: R1.2, U$5.24
- new net 1TO2: U$5.DOUT, U$6.DIN
- new net 2TO3: U$6.DOUT, U$7.DIN
- new net 3TO4: U$7.DOUT, U$8.DIN
- new net ANT: C17.2, C18.2, Y2.FEED
- new net IR_SENSOR: U$1.P$2, U$3.22
- new net N$1: C5.2, R1.1, U$2.SIG
- new net N$15: C12.1, Q2.1, R9.1, U4.9
- new net N$17: L5.1, L7.2, U4.13
- new net N$18: C15.1, C16.1, L6.1, U4.11
- new net N$19: R10.1, U4.16
- new net N$2: R2.2, U$1.P$1
- new net N$20: C14.1, U4.19
- new net N$21: L6.2, L7.1, U4.12
- new net N$22: C18.1, L5.2
- new net N$3: C5.1, R3.1
- new net N$4: R3.2, R4.1, U1.1
- new net N$5: C2.1, L1.2, RECEIVER.VCC
- new net N$6: R4.2, U1.2, U1.3
- new net PIN3: TRANSMITTER.SIGNAL
- new net SIGNAL_DET: R5.2, U$3.6
- new net SPDIF_IN_1: U1.4, U2.3
- new net SPDIF_IN_2: R5.1, RECEIVER.SIGNAL, U2.1
- new net TEENSY_SPDIF_IN: U$3.14, U2.4
- new net WS2812B_DIN: U$5.DIN, U3.4
- net 3V3: now also C1.1, C3.1, L1.1, R2.1, TRANSMITTER.VCC, U$3.3.3V, U$9.2, U1.14, U2.5, U4.15, U4.18, U4.7; no longer M1.2, U$2.VCC, U$3.VCC, U$5.3.3V, U1.5
- net 5V: now also C4.1, C6.1, C7.1, C8.1, J1.VBUS, U$3.VIN, U$5.VDD, U$6.VDD, U$7.VDD, U$8.VDD, U3.5; no longer U$5.VIN
- net CE: now also U$3.5, U$9.3, U4.1; no longer M1.3, U$5.5
- net CSN: now also U$3.9, U$9.4, U4.2; no longer M1.4, U$5.9
- net GND: now also C1.2, C12.2, C13.2, C14.2, C15.2, C16.2, C17.1, C2.2, C3.2, C4.2, C6.2, C7.2, C8.2, J1.GND, R1.2, R10.2, R6.1, RECEIVER.GND, TRANSMITTER.GND, U$1.P$3, U$2.GND1, U$2.GND2, U$2.GND3, U$3.AGND, U$3.GND2, U$5.VSS, U$6.VSS, U$7.VSS, U$8.VSS, U$9.1, U1.7, U2.2, U3.1, U3.3, U4.0, U4.14, U4.17, U4.20, U4.8; no longer M1.1, U$2.GND, U$5.AGND, U$5.GND, U$5.GND2, U1.2
- net I2S_DIN: now also U$3.8; no longer U$5.8
- net I2S_DOUT: now also U$3.7; no longer U$5.7
- net IRQ: now also U$3.16, U$9.8, U4.6; no longer M1.8, U$5.16
- net LED: now also U$3.3, U3.2; no longer U$5.3
- net LRCLK: now also U$3.20; no longer U$5.20
- net MCLK: now also U$3.23; no longer U$5.23
- net MISO: now also U$3.12, U$9.7, U4.5; no longer M1.7, U$5.12
- net MOSI: now also U$3.11, U$9.6, U4.4; no longer M1.6, U$5.11
- net MUX_SWITCH: now also R6.2, U$3.4, U2.6; no longer U$5.25, U1.6
- net N$16: now also C13.1, Q2.3, R9.2, U4.10; no longer U$5.17
- net ON/OFF: now also U$3.ON/OFF; no longer U$5.ON/OFF
- net S/PDIF-OUT: now also U$3.15; no longer U$3.SIGNAL, U$5.15
- net SCK: now also U$3.13, U$9.5, U4.3; no longer M1.5, U$5.13
- net SCLK: now also U$3.21; no longer U$5.21
- net SGTL_SCL: now also U$3.19; no longer U$5.19
- net SGTL_SDA: now also U$3.18; no longer U$5.18
Routing:
- net 5V: track 0.00 -> 113.4 mm
- net 3V3: track 0.00 -> 95.8 mm, vias 0 -> 2
- net CE: track 0.00 -> 60.7 mm
- net MUX_SWITCH: track 0.00 -> 56.6 mm
- net IR_SENSOR: track 0.00 -> 51.0 mm
- net LED: track 0.00 -> 47.0 mm
- net SPDIF_IN_2: track 0.00 -> 31.8 mm, vias 0 -> 1
- net CSN: track 0.00 -> 29.9 mm, vias 0 -> 1
- net IRQ: track 0.00 -> 25.8 mm
- net SPDIF_IN_1: track 0.00 -> 21.6 mm, vias 0 -> 1
- net SCK: track 0.00 -> 19.1 mm
- net WS2812B_DIN: track 0.00 -> 19.0 mm
- net MOSI: track 0.00 -> 16.4 mm
- net MISO: track 0.00 -> 13.7 mm
- net 2TO3: track 0.00 -> 11.0 mm
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- added copper zone on layer 1, net GND
- added copper zone on layer 16, net GND
Other:
- board outline added: 66 x 44.5 mm
